Commit message: Modified aruco single.launch to obtainb correct camera position, updated the camera sensor plugin, now attached to the ee, added new package for panda_control using active inference, changed publishing rate for the /joint_states to match the one in the real robot i.e. 1khz. Succesfully coded free-energy minimization using only proprioceptive sensors i.e. encoders in static situation

File: franka_description/robots/panda_arm_camera.urdf.xacro (robot description, xacro)
@@ -8,5 +8,5 @@
   <xacro:include filename="$(find franka_description)/robots/panda_camera.gazebo.xacro"/>
   <xacro:panda_arm />
-  <xacro:panda_camera />
+  <xacro:panda_camera connected_to="panda_link8"/>
   <xacro:panda_gazebo robot_name="$(arg robot_name)" />
   <xacro:panda_camera_gazebo />

File: franka_description/robots/panda_camera.gazebo.xacro (robot description, xacro)
@@ -21,10 +21,10 @@
 	      	<plugin name="camera_controller" filename="libgazebo_ros_camera.so">
 			<alwaysOn>true</alwaysOn>
-			<updateRate>0.0</updateRate>
+			<updateRate>30.0</updateRate>
 			<cameraName>panda/camera1</cameraName>
 			<imageTopicName>image_raw</imageTopicName>
 			<cameraInfoTopicName>camera_info</cameraInfoTopicName>
 			<frameName>camera</frameName>
-			<hackBaseline>0.07</hackBaseline>
+			<hackBaseline>0.0</hackBaseline>
 			<distortionK1>0.0</distortionK1>
 			<distortionK2>0.0</distortionK2>

File: franka_description/robots/panda_camera.xacro (robot description, xacro)
@@ -1,7 +1,13 @@
 <?xml version="1.0" encoding="utf-8"?>
-<robot xmlns:xacro="http://www.ros.org/wiki/xacro" name="panda">
-  <xacro:macro name="panda_camera">
+<robot xmlns:xacro="http://www.ros.org/wiki/xacro" name="camera">
+  <xacro:macro name="panda_camera" params="connected_to:='' ">
     <xacro:property name="cameraSize" value="0.05"/>
     <xacro:property name="cameraMass" value="0.1"/>
+   <joint name="camera_joint" type="fixed">
+     <axis xyz="0 0 0" />
+     <origin xyz="0 0 0" rpy="0 -1.581 0"/>
+     <parent link="${connected_to}"/>
+     <child link="camera_link"/>
+   </joint>
    <link name="camera_link">
     <collision>
@@ -14,5 +20,5 @@
       <origin xyz="0 0 0" rpy="0 0 0"/>
       <geometry>
-        <box size="${cameraSize} ${cameraSize} ${cameraSize}"/>
+        <box size="${cameraSize} ${0.5*cameraSize} ${0.5*cameraSize}"/>
       </geometry>
       <material name="green"/>
@@ -25,10 +31,4 @@
     </inertial>
   </link>
-  <joint name="camera_joint" type="fixed">
-    <axis xyz="0 1 0" />
-    <origin xyz="1 0 1" rpy="0 1.578 0"/>
-    <parent link="panda_link0"/>
-    <child link="camera_link"/>
-  </joint>
   </xacro:macro>
 </robot>
