Commit message: Modified mesh files of the robot arm for better visualization and added marker .dae

File: franka_description/robots/panda.gazebo.xacro (robot description, xacro)
@@ -4,5 +4,4 @@
         <!-- Link0 -->
         <gazebo reference="${robot_name}_link0">
-            <material>Gazebo/Grey</material>
             <mu1>0.2</mu1>
             <mu2>0.2</mu2>
@@ -10,5 +9,4 @@
         <!-- Link1 -->
         <gazebo reference="${robot_name}_link1">
-            <material>Gazebo/White</material>
             <mu1>0.2</mu1>
             <mu2>0.2</mu2>
@@ -16,5 +14,4 @@
         <!-- Link2 -->
         <gazebo reference="${robot_name}_link2">
-            <material>Gazebo/White</material>
             <mu1>0.2</mu1>
             <mu2>0.2</mu2>
@@ -22,5 +19,4 @@
         <!-- Link3 -->
         <gazebo reference="${robot_name}_link3">
-            <material>Gazebo/White</material>
             <mu1>0.2</mu1>
             <mu2>0.2</mu2>
@@ -28,5 +24,4 @@
         <!-- Link4 -->
         <gazebo reference="${robot_name}_link4">
-            <material>Gazebo/White</material>
             <mu1>0.2</mu1>
             <mu2>0.2</mu2>
@@ -34,5 +29,4 @@
         <!-- Link5 -->
         <gazebo reference="${robot_name}_link5">
-            <material>Gazebo/White</material>
             <mu1>0.2</mu1>
             <mu2>0.2</mu2>
@@ -40,5 +34,4 @@
         <!-- Link6 -->
         <gazebo reference="${robot_name}_link6">
-            <material>Gazebo/White</material>
             <mu1>0.2</mu1>
             <mu2>0.2</mu2>
@@ -46,5 +39,4 @@
         <!-- Link7 -->
         <gazebo reference="${robot_name}_link7">
-            <material>Gazebo/Grey</material>
             <mu1>0.2</mu1>
             <mu2>0.2</mu2>
@@ -52,5 +44,4 @@
         <!-- Link8 -->
         <gazebo reference="${robot_name}_link8">
-            <material>Gazebo/Grey</material>
             <mu1>0.2</mu1>
             <mu2>0.2</mu2>
@@ -58,5 +49,4 @@
         <!-- LinkHand -->
         <gazebo reference="${robot_name}_hand">
-            <material>Gazebo/Grey</material>
             <mu1>0.2</mu1>
             <mu2>0.2</mu2>
@@ -64,5 +54,4 @@
         <!-- LinkRightFinger -->
         <gazebo reference="${robot_name}_rightfinger">
-            <material>Gazebo/Grey</material>
             <mu1>0.2</mu1>
             <mu2>0.2</mu2>
@@ -70,5 +59,4 @@
         <!-- LinkLeftFinger -->
         <gazebo reference="${robot_name}_leftfinger">
-            <material>Gazebo/Grey</material>
             <mu1>0.2</mu1>
             <mu2>0.2</mu2>

File: franka_description/robots/panda_arm.xacro (robot description, xacro)
@@ -231,4 +231,16 @@
       <axis xyz="0 0 0"/>
     </joint>
+    <link name="marker_link">
+    <visual>
+      <geometry>
+          <mesh filename="package://${description_pkg}/meshes/visual/marker.dae" scale="1 1 0.001"/>
+      </geometry>
+    </visual>
+  </link>
+  <joint name="marker_joint" type="fixed">
+    <origin rpy="0 0 ${-pi/2}" xyz="0.75 0 0"/>
+    <parent link="panda_link0"/>
+    <child link="marker_link"/>
+  </joint>
   </xacro:macro>
 </robot>

File: franka_description/robots/panda_arm_camera.urdf.xacro (robot description, xacro)
@@ -8,5 +8,5 @@
   <xacro:include filename="$(find franka_description)/robots/panda_camera.gazebo.xacro"/>
   <xacro:panda_arm />
-  <xacro:panda_camera connected_to="panda_link8"/>
+  <xacro:panda_camera connected_to="panda_link8" rpy="${pi} ${-pi/2} 0" xyz="0 0 0"/>
   <xacro:panda_gazebo robot_name="$(arg robot_name)" />
   <xacro:panda_camera_gazebo />

File: franka_description/robots/panda_camera.xacro (robot description, xacro)
@@ -1,10 +1,10 @@
 <?xml version="1.0" encoding="utf-8"?>
 <robot xmlns:xacro="http://www.ros.org/wiki/xacro" name="camera">
-  <xacro:macro name="panda_camera" params="connected_to:='' ">
+  <xacro:macro name="panda_camera" params="connected_to:='' rpy:='' xyz:=''">
     <xacro:property name="cameraSize" value="0.05"/>
     <xacro:property name="cameraMass" value="0.1"/>
    <joint name="camera_joint" type="fixed">
      <axis xyz="0 0 0" />
-     <origin xyz="0 0 0" rpy="0 -1.581 0"/>
+       <origin xyz="${xyz}" rpy="${rpy}"/>
      <parent link="${connected_to}"/>
      <child link="camera_link"/>
