Commit message: Solved problems with Gazebo GUI, cleaned xacros, added aruco_ros, added camera, added aruco_marker

File: franka_description/robots/panda.transmission.xacro (robot description, xacro)
@@ -6,4 +6,5 @@
             <plugin name="gazebo_ros_control" filename="libgazebo_ros_control.so">
                 <!-- <robotNamespace>/${robot_name}</robotNamespace> -->
+ 		<legacyModeNS>true</legacyModeNS>
             </plugin>
         </gazebo>
@@ -78,24 +79,4 @@
             </actuator>
         </transmission>
-        <transmission name="${robot_name}_leftfinger">
-            <type>transmission_interface/SimpleTransmission</type>
-            <joint name="${robot_name}_finger_joint1">
-                <hardwareInterface>hardware_interface/EffortJointInterface</hardwareInterface>
-            </joint>
-            <actuator name="${robot_name}_finger_joint1">
-                <hardwareInterface>hardware_interface/EffortJointInterface</hardwareInterface>
-                <mechanicalReduction>1</mechanicalReduction>
-            </actuator>
-        </transmission>
-        <transmission name="${robot_name}_rightfinger">
-            <type>transmission_interface/SimpleTransmission</type>
-            <joint name="${robot_name}_finger_joint2">
-                <hardwareInterface>hardware_interface/EffortJointInterface</hardwareInterface>
-            </joint>
-            <actuator name="${robot_name}_finger_joint2">
-                <hardwareInterface>hardware_interface/EffortJointInterface</hardwareInterface>
-                <mechanicalReduction>1</mechanicalReduction>
-            </actuator>
-        </transmission>
     </xacro:macro>
 </robot>

File: franka_description/robots/panda_arm.xacro (robot description, xacro)
@@ -10,4 +10,6 @@
     </xacro:unless>
     <xacro:property name="joint_damping" value="1.0"/>
+    <xacro:property name="cameraSize" value="0.05"/>
+    <xacro:property name="cameraMass" value="0.1"/>
     <link name="world" />
     <joint name="robot_to_world" type="fixed">

File: franka_description/robots/panda_arm_camera.urdf.xacro (robot description, xacro)
@@ -3,10 +3,12 @@
   <xacro:arg name="robot_name" default="panda"/>
   <xacro:include filename="$(find franka_description)/robots/panda_arm.xacro"/>
-  <xacro:include filename="$(find franka_description)/robots/hand.xacro"/>
   <xacro:include filename="$(find franka_description)/robots/panda.gazebo.xacro"/>
   <xacro:include filename="$(find franka_description)/robots/panda.transmission.xacro"/>
+  <xacro:include filename="$(find franka_description)/robots/panda_camera.xacro"/>
+  <xacro:include filename="$(find franka_description)/robots/panda_camera.gazebo.xacro"/>
   <xacro:panda_arm />
-  <xacro:hand ns="panda" rpy="0 0 ${-pi/4}" connected_to="panda_link8"/>
+  <xacro:panda_camera />
   <xacro:panda_gazebo robot_name="$(arg robot_name)" />
+  <xacro:panda_camera_gazebo />
   <xacro:panda_transmission robot_name="$(arg robot_name)" />
 </robot>

Commit message: Added forward dynamics and set up structure for adding visual data as in the Matlab code using FK. Still missing the correct use of the camera Gazebo plugin

File: franka_description/robots/panda.transmission.xacro (robot description, xacro)
@@ -79,4 +79,14 @@
             </actuator>
         </transmission>
+        <transmission name="${robot_name}_tran_8">
+            <type>transmission_interface/SimpleTransmission</type>
+            <joint name="${robot_name}_joint8">
+                <hardwareInterface>hardware_interface/EffortJointInterface</hardwareInterface>
+            </joint>
+            <actuator name="${robot_name}_motor_8">
+                <hardwareInterface>hardware_interface/EffortJointInterface</hardwareInterface>
+                <mechanicalReduction>1</mechanicalReduction>
+            </actuator>
+        </transmission>
     </xacro:macro>
 </robot>

File: franka_description/robots/panda_arm.xacro (robot description, xacro)
@@ -10,6 +10,4 @@
     </xacro:unless>
     <xacro:property name="joint_damping" value="1.0"/>
-    <xacro:property name="cameraSize" value="0.05"/>
-    <xacro:property name="cameraMass" value="0.1"/>
     <link name="world" />
     <joint name="robot_to_world" type="fixed">
@@ -221,15 +219,17 @@
       <inertial>
         <origin xyz="0 0 0" rpy="0 0 0"/>
-        <mass value="0.0"/>
-        <inertia ixx="0.3" ixy="0.0" ixz="0.0" iyy="0.3" iyz="0.0" izz="0.3"/>
-      </inertial>
-    </link>
-    <joint name="${arm_id}_joint8" type="fixed">
+        <mass value="0.001"/>
+        <inertia ixx="0.3" ixy="0.0" ixz="0.0" iyy="0.3" iyz="0.0" izz="0.3"/>
+      </inertial>
+    </link>
+    <joint name="${arm_id}_joint8" type="revolute">
       <origin rpy="0 0 0" xyz="0 0 0.107"/>
       <parent link="${arm_id}_link7"/>
       <child link="${arm_id}_link8"/>
-      <axis xyz="0 0 0"/>
-    </joint>
-    <link name="marker_link">
+      <axis xyz="0 0 1"/>
+      <limit effort="1" lower="0" upper="0.1" velocity="0.1"/>
+      <dynamics damping="100"/>
+    </joint>
+    <!--link name="marker_link">
     <visual>
       <geometry>
@@ -239,8 +239,8 @@
   </link>
   <joint name="marker_joint" type="fixed">
-    <origin rpy="0 0 ${-pi/2}" xyz="0.75 0 0"/>
+    <origin rpy="0 0 ${-pi/2}" xyz="-0.75 0 0"/>
     <parent link="panda_link0"/>
     <child link="marker_link"/>
-  </joint>
+  </joint-->
   </xacro:macro>
 </robot>

File: franka_description/robots/panda_arm_camera.urdf.xacro (robot description, xacro)
@@ -3,10 +3,10 @@
   <xacro:arg name="robot_name" default="panda"/>
   <xacro:include filename="$(find franka_description)/robots/panda_arm.xacro"/>
+  <xacro:include filename="$(find franka_description)/robots/panda_camera.xacro"/>
   <xacro:include filename="$(find franka_description)/robots/panda.gazebo.xacro"/>
   <xacro:include filename="$(find franka_description)/robots/panda.transmission.xacro"/>
-  <xacro:include filename="$(find franka_description)/robots/panda_camera.xacro"/>
   <xacro:include filename="$(find franka_description)/robots/panda_camera.gazebo.xacro"/>
   <xacro:panda_arm />
-  <xacro:panda_camera connected_to="panda_link8" rpy="${pi} ${-pi/2} 0" xyz="0 0 0"/>
+  <xacro:panda_camera ns="panda" connected_to="panda_link8" rpy="${pi} ${-pi/2} 0" xyz="0 0 0"/>
   <xacro:panda_gazebo robot_name="$(arg robot_name)" />
   <xacro:panda_camera_gazebo />

File: franka_description/robots/panda_camera.gazebo.xacro (robot description, xacro)
@@ -3,5 +3,5 @@
   <xacro:macro name="panda_camera_gazebo">
  <!-- Camera -->
-    <gazebo reference="camera_link">
+    <gazebo reference="panda_camera">
     	<material>Gazebo/Green</material>
 	    	<sensor type="camera" name="camera1">
@@ -25,5 +25,6 @@
 			<imageTopicName>image_raw</imageTopicName>
 			<cameraInfoTopicName>camera_info</cameraInfoTopicName>
-			<frameName>camera</frameName>
+			<frameName>panda_camera_frame</frameName>
+      <broadcastTF>true</broadcastTF>
 			<hackBaseline>0.0</hackBaseline>
 			<distortionK1>0.0</distortionK1>

File: franka_description/robots/panda_camera.urdf.xacro (robot description, xacro)
@@ -2,4 +2,4 @@
 <robot xmlns:xacro="http://www.ros.org/wiki/xacro" name="panda_camera">
   <xacro:include filename="panda_camera.xacro"/>
-  <xacro:panda_camera />
+  <xacro:panda_camera ns="panda"/>
 </robot>

File: franka_description/robots/panda_camera.xacro (robot description, xacro)
@@ -1,32 +1,29 @@
 <?xml version="1.0" encoding="utf-8"?>
-<robot xmlns:xacro="http://www.ros.org/wiki/xacro" name="camera">
-  <xacro:macro name="panda_camera" params="connected_to:='' rpy:='' xyz:=''">
-    <xacro:property name="cameraSize" value="0.05"/>
-    <xacro:property name="cameraMass" value="0.1"/>
-   <joint name="camera_joint" type="fixed">
-     <axis xyz="0 0 0" />
-       <origin xyz="${xyz}" rpy="${rpy}"/>
-     <parent link="${connected_to}"/>
-     <child link="camera_link"/>
-   </joint>
-   <link name="camera_link">
-    <collision>
-      <origin xyz="0 0 0" rpy="0 0 0"/>
+<robot xmlns:xacro="http://www.ros.org/wiki/xacro" name="panda_camera">
+  <xacro:macro name="panda_camera" params="connected_to:='' ns:='' rpy:='' xyz:='' ">
+  <xacro:unless value="${connected_to == ''}">
+    <joint name="${ns}_camera_joint" type="fixed">
+      <parent link="${connected_to}"/>
+      <child link="${ns}_camera"/>
+      <origin xyz="${xyz}" rpy="${rpy}"/>
+    </joint>
+  </xacro:unless>
+  <xacro:property name="cameraSize" value="0.05"/>
+  <link name="${ns}_camera">
+    <visual>
       <geometry>
-        <box size="${cameraSize} ${cameraSize} ${cameraSize}"/>
-      </geometry>
-    </collision>
-    <visual>
-      <origin xyz="0 0 0" rpy="0 0 0"/>
-      <geometry>
-        <box size="${cameraSize} ${0.5*cameraSize} ${0.5*cameraSize}"/>
+          <box size="${cameraSize} ${0.5*cameraSize} ${0.5*cameraSize}"/>
       </geometry>
       <material name="green"/>
     </visual>
+    <collision>
+      <geometry>
+          <box size="${cameraSize} ${0.5*cameraSize} ${0.5*cameraSize}"/>
+      </geometry>
+    </collision>
     <inertial>
-      <mass value="${cameraMass}" />
       <origin xyz="0 0 0" rpy="0 0 0"/>
-      <box_inertia m="${cameraMass}" x="${cameraSize}" y="${cameraSize}" z="${cameraSize}" />
-      <inertia ixx="1e-6" ixy="0" ixz="0" iyy="1e-6" iyz="0" izz="1e-6" />
+      <mass value="0.1"/>
+      <inertia ixx="0.01" ixy="0.0" ixz="0.0" iyy="0.01" iyz="0.0" izz="0.01"/>
     </inertial>
   </link>
