Commit message: Simplified packages and simulation. Added fixed camera and marker on the end-effector. Published beliefs about the states in a ROS topic in the class AIC.cpp

File: franka_description/robots/panda_arm.xacro (robot description, xacro)
@@ -231,5 +231,5 @@
       <dynamics damping="100"/>
     </joint>
-    <!--link name="marker_link">
+    <link name="marker_link">
     <visual>
       <geometry>
@@ -239,8 +239,8 @@
   </link>
   <joint name="marker_joint" type="fixed">
-    <origin rpy="0 0 ${-pi/2}" xyz="-0.75 0 0"/>
-    <parent link="panda_link0"/>
+    <origin rpy="0 0 0" xyz="0 0 0.0011"/>
+    <parent link="panda_link8"/>
     <child link="marker_link"/>
-  </joint-->
+  </joint>
   </xacro:macro>
 </robot>

File: franka_description/robots/panda_arm_camera.urdf.xacro (robot description, xacro)
@@ -8,5 +8,7 @@
   <xacro:include filename="$(find franka_description)/robots/panda_camera.gazebo.xacro"/>
   <xacro:panda_arm />
-  <xacro:panda_camera ns="panda" connected_to="panda_link8" rpy="${pi} ${-pi/2} 0" xyz="0 0 0"/>
+  <xacro:panda_camera ns="panda" connected_to="world" rpy="0 ${-pi/3} ${pi}" xyz="1 0 0.05"/>
+  <!--Other frame with possible use with Aruco, this has the z pointing to the image-->
+  <!--xacro:panda_camera ns="camera_ref" connected_to="world" rpy="0 ${-pi/3+pi/2} ${pi}" xyz="1 0 0.05"/-->
   <xacro:panda_gazebo robot_name="$(arg robot_name)" />
   <xacro:panda_camera_gazebo />

File: franka_description/robots/panda_camera.gazebo.xacro (robot description, xacro)
@@ -25,5 +25,8 @@
 			<imageTopicName>image_raw</imageTopicName>
 			<cameraInfoTopicName>camera_info</cameraInfoTopicName>
-			<frameName>panda_camera_frame</frameName>
+			<frameName>panda_optical_frame</frameName>
+      <CxPrime>1224.5</CxPrime>
+      <Cx>1224.5</Cx>
+      <Cy>1025.5</Cy>
       <broadcastTF>true</broadcastTF>
 			<hackBaseline>0.0</hackBaseline>

File: franka_description/robots/panda_camera.xacro (robot description, xacro)
@@ -28,4 +28,11 @@
     </inertial>
   </link>
+  <!--joint name="${ns}_optical_joint" type="fixed">
+      <origin xyz="0 0 0" rpy="${-pi/2} 0.0 ${-pi/2}" />
+      <parent link="${ns}_camera" />
+      <child link="${ns}_optical_frame"/>
+    </joint>
+    <link name="${ns}_optical_frame">
+    </link-->
   </xacro:macro>
 </robot>

Commit message: Added boxes and pick and place cycle for the AIC and MRAC.

File: franka_description/robots/panda_arm.xacro (robot description, xacro)
@@ -10,5 +10,4 @@
     </xacro:unless>
     <xacro:property name="joint_damping" value="1.0"/>
-    <link name="world" />
     <joint name="robot_to_world" type="fixed">
       <parent link="world" />
@@ -231,5 +230,5 @@
       <dynamics damping="100"/>
     </joint>
-    <link name="marker_link">
+    <!--link name="marker_link">
     <visual>
       <geometry>
@@ -242,5 +241,5 @@
     <parent link="panda_link8"/>
     <child link="marker_link"/>
-  </joint>
+  </joint-->
   </xacro:macro>
 </robot>

File: franka_description/robots/panda_arm_camera.urdf.xacro (robot description, xacro)
@@ -2,15 +2,46 @@
 <robot xmlns:xacro="http://www.ros.org/wiki/xacro" name="panda">
   <xacro:arg name="robot_name" default="panda"/>
+  <!-- Empty link to referr everything to -->
+  <link name="world" />
+  <!-- Robot arm -->
   <xacro:include filename="$(find franka_description)/robots/panda_arm.xacro"/>
-  <xacro:include filename="$(find franka_description)/robots/panda_camera.xacro"/>
   <xacro:include filename="$(find franka_description)/robots/panda.gazebo.xacro"/>
   <xacro:include filename="$(find franka_description)/robots/panda.transmission.xacro"/>
-  <xacro:include filename="$(find franka_description)/robots/panda_camera.gazebo.xacro"/>
+  <!-- Robot1 Pedestal -->
+  <xacro:include filename="$(find franka_description)/robots/robot_pedestal/robot_pedestal.urdf.xacro"/>
+  <xacro:robot_pedestal_urdf pedestal_prefix="robot1_" pedestal_parent="world" pedestal_height="0.3">
+    <origin xyz="0.3 -0.5 0.0" rpy="0 0 0"/>
+  </xacro:robot_pedestal_urdf>
+  <!-- Camera-->
+  <!--xacro:include filename="$(find franka_description)/robots/panda_camera.xacro"/>
+  <xacro:include filename="$(find franka_description)/robots/panda_camera.gazebo.xacro"/-->
+  <!-- bins -->
+  <xacro:include filename="$(find franka_description)/robots/bin/bin.urdf.xacro"/>
+  <xacro:bin_urdf prefix="bin_1_"/>
+  <xacro:bin_urdf prefix="bin_2_"/>
+  <!-- Robot arm definition-->
   <xacro:panda_arm />
-  <xacro:panda_camera ns="panda" connected_to="world" rpy="0 ${-pi/3} ${pi}" xyz="1 0 0.05"/>
-  <!--Other frame with possible use with Aruco, this has the z pointing to the image-->
-  <!--xacro:panda_camera ns="camera_ref" connected_to="world" rpy="0 ${-pi/3+pi/2} ${pi}" xyz="1 0 0.05"/-->
   <xacro:panda_gazebo robot_name="$(arg robot_name)" />
-  <xacro:panda_camera_gazebo />
   <xacro:panda_transmission robot_name="$(arg robot_name)" />
+  <!-- Camera definition-->
+  <!--xacro:panda_camera ns="panda" connected_to="world" rpy="0 ${-pi/3} ${pi}" xyz="1 0 0.05"/>
+  <xacro:panda_camera_gazebo /-->
+  <!-- pedestal to world -->
+  <joint name="robot1_pedestal_to_world_interface" type="fixed">
+    <parent link="world" />
+    <child link="robot1_pedestal_link" />
+    <origin xyz="0.4 -0.6 0.0" rpy="0.0 0.0 0.0"/>
+  </joint>
+  <!-- bin 1 -->
+  <joint name="bin_1_joint" type="fixed">
+    <parent link="world" />
+    <child link="bin_1_base_link" />
+    <origin xyz="0.3 0.55 0" rpy="0 0 0" />
+  </joint>
+  <!-- bin 2 -->
+  <joint name="bin_2_joint" type="fixed">
+    <parent link="world" />
+    <child link="bin_2_base_link" />
+    <origin xyz="0.4 -0.6 0.3" rpy="0 0 0" />
+  </joint>
 </robot>

File: franka_description/robots/panda_camera.gazebo.xacro (robot description, xacro)
@@ -26,14 +26,13 @@
 			<cameraInfoTopicName>camera_info</cameraInfoTopicName>
 			<frameName>panda_optical_frame</frameName>
-      <CxPrime>1224.5</CxPrime>
-      <Cx>1224.5</Cx>
-      <Cy>1025.5</Cy>
+      <Cx>0</Cx>
+      <Cy>0</Cy>
       <broadcastTF>true</broadcastTF>
 			<hackBaseline>0.0</hackBaseline>
-			<distortionK1>0.0</distortionK1>
-			<distortionK2>0.0</distortionK2>
-			<distortionK3>0.0</distortionK3>
-			<distortionT1>0.0</distortionT1>
-			<distortionT2>0.0</distortionT2>
+			<distortionK1>0.000000001</distortionK1>
+			<distortionK2>0.000000001</distortionK2>
+			<distortionK3>0.000000001</distortionK3>
+			<distortionT1>0.000000001</distortionT1>
+			<distortionT2>0.000000001</distortionT2>
 	      	</plugin>
     	</sensor>

Commit message: Improved simulation environment. Added inertia tensor from meshlab for the real robot, changed the masses and the friction also

File: franka_description/robots/panda_arm.xacro (robot description, xacro)
@@ -1,4 +1,41 @@
 <?xml version='1.0' encoding='utf-8'?>
 <robot xmlns:xacro="http://www.ros.org/wiki/xacro" name="panda">
+  <!-- This masses are incorrect on purpose, off by 20% w.r.t the model-->
+  <xacro:property name="mass_link0" value="3.66357" />
+  <xacro:property name="mass_link1" value="2.04471" />
+  <xacro:property name="mass_link2" value="2.56414" />
+  <xacro:property name="mass_link3" value="2.48050" />
+  <xacro:property name="mass_link4" value="2.02754" />
+  <xacro:property name="mass_link5" value="3.09611" />
+  <xacro:property name="mass_link6" value="1.66736" />
+  <xacro:property name="mass_link7" value="0.75606" />
+  <xacro:property name="mass_link8" value="0.1" />
+  <xacro:property name="link0_cog" value="-0.029190 -0.000879 0.056603" />
+  <xacro:property name="link1_cog" value="0.000011 -0.031266 -0.069373" />
+  <xacro:property name="link2_cog" value="-0.000013 -0.070322 0.031178" />
+  <xacro:property name="link3_cog" value="0.044348 0.024928 -0.038130" />
+  <xacro:property name="link4_cog" value="-0.038550 0.039526 0.024716" />
+  <xacro:property name="link5_cog" value="-0.000064 0.038412 -0.109970" />
+  <xacro:property name="link6_cog" value="0.051002 0.006933 0.006169" />
+  <xacro:property name="link7_cog" value="0.010361 0.010360 0.079108" />
+  <!-- Correct masses
+  <xacro:property name="mass_link0" value="3.06357" />
+  <xacro:property name="mass_link1" value="2.34471" />
+  <xacro:property name="mass_link2" value="2.36414" />
+  <xacro:property name="mass_link3" value="2.38050" />
+  <xacro:property name="mass_link4" value="2.42754" />
+  <xacro:property name="mass_link5" value="3.49611" />
+  <xacro:property name="mass_link6" value="1.46736" />
+  <xacro:property name="mass_link7" value="0.45606" />
+  <xacro:property name="mass_link8" value="0.001" /> -->
+    <xacro:macro name="cylinder_inertial" params="radius length mass *origin">
+      <inertial>
+        <mass value="${mass}" />
+        <xacro:insert_block name="origin" />
+        <inertia ixx="${0.0833333 * mass * (3 * radius * radius + length * length)}" ixy="0.0" ixz="0.0"
+          iyy="${0.0833333 * mass * (3 * radius * radius + length * length)}" iyz="0.0"
+          izz="${0.5 * mass * radius * radius}" />
+      </inertial>
+  </xacro:macro>
   <xacro:macro name="panda_arm" params="arm_id:='panda' description_pkg:='franka_description' connected_to:='' xyz:='0 0 0' rpy:='0 0 0'">
     <xacro:unless value="${not connected_to}">
@@ -28,7 +65,7 @@
       </collision>
       <inertial>
-        <origin xyz="0 0 0" rpy="0 0 0"/>
-        <mass value="3.06"/>
-        <inertia ixx="0.3" ixy="0.0" ixz="0.0" iyy="0.3" iyz="0.0" izz="0.3"/>
+        <origin xyz="${link0_cog}" rpy="0 0 0"/>
+        <mass value="${mass_link0}"/>
+        <inertia ixx="0.009" iyy="0.0122" izz="0.0122" ixy="0.0" ixz="-0.00010" iyz="0.0"/>
       </inertial>
     </link>
@@ -45,7 +82,7 @@
       </collision>
       <inertial>
-        <origin xyz="0 0 0" rpy="0 0 0"/>
-        <mass value="2.34"/>
-        <inertia ixx="0.3" ixy="0.0" ixz="0.0" iyy="0.3" iyz="0.0" izz="0.3"/>
+        <origin xyz="${link1_cog}" rpy="0 0 0"/>
+        <mass value="${mass_link1}"/>
+        <inertia ixx="0.01418" iyy="0.01181" izz="0.005515" ixy="0.0" ixz="0.0" iyz="0.00236"/>
       </inertial>
     </link>
@@ -71,7 +108,7 @@
       </collision>
       <inertial>
-        <origin xyz="0 0 0" rpy="0 0 0"/>
-        <mass value="2.36"/>
-        <inertia ixx="0.3" ixy="0.0" ixz="0.0" iyy="0.3" iyz="0.0" izz="0.3"/>
+        <origin xyz="${link2_cog}" rpy="0 0 0"/>
+        <mass value="${mass_link2}"/>
+        <inertia ixx="0.014" ixy="0.0" ixz="0.0" iyy="0.0055" iyz="-0.0023" izz="0.01259"/>
       </inertial>
     </link>
@@ -97,7 +134,7 @@
       </collision>
       <inertial>
-        <origin xyz="0 0 0" rpy="0 0 0"/>
-        <mass value="2.38"/>
-        <inertia ixx="0.3" ixy="0.0" ixz="0.0" iyy="0.3" iyz="0.0" izz="0.3"/>
+        <origin xyz="${link3_cog}" rpy="0 0 0"/>
+        <mass value="${mass_link3}"/>
+        <inertia ixx="0.00716" ixy="-0.00102" ixz="-0.02040" iyy="0.00920" iyz="-0.00102" izz="0.007159"/>
       </inertial>
     </link>
@@ -123,7 +160,7 @@
       </collision>
       <inertial>
-        <origin xyz="0 0 0" rpy="0 0 0"/>
-        <mass value="2.43"/>
-        <inertia ixx="0.3" ixy="0.0" ixz="0.0" iyy="0.3" iyz="0.0" izz="0.3"/>
+        <origin xyz="${link4_cog}" rpy="0 0 0"/>
+        <mass value="${mass_link4}"/>
+        <inertia ixx="0.008164" ixy="0.003061" ixz="0.00102" iyy="0.008165" iyz="0.00102" izz="0.009185"/>
       </inertial>
     </link>
@@ -149,7 +186,7 @@
       </collision>
       <inertial>
-        <origin xyz="0 0 0" rpy="0 0 0"/>
-        <mass value="3.5"/>
-        <inertia ixx="0.3" ixy="0.0" ixz="0.0" iyy="0.3" iyz="0.0" izz="0.3"/>
+        <origin xyz="${link5_cog}" rpy="0 0 0"/>
+        <mass value="${mass_link5}"/>
+        <inertia ixx="0.0307" ixy="0.0" ixz="0.0" iyy="0.02761" iyz="-0.0613" izz="0.00818"/>
       </inertial>
     </link>
@@ -175,7 +212,7 @@
       </collision>
       <inertial>
-        <origin xyz="0 0 0" rpy="0 0 0"/>
-        <mass value="1.47"/>
-        <inertia ixx="0.3" ixy="0.0" ixz="0.0" iyy="0.3" iyz="0.0" izz="0.3"/>
+        <origin xyz="${link6_cog}" rpy="0 0 0"/>
+        <mass value="${mass_link6}"/>
+        <inertia ixx="0.00205" ixy="0.0" ixz="0.0" iyy="0.004089" iyz="0" izz="0.00490"/>
       </inertial>
     </link>
@@ -202,5 +239,5 @@
       <inertial>
         <origin xyz="0 0 0" rpy="0 0 0"/>
-        <mass value="0.45"/>
+        <mass value="${mass_link7}"/>
         <inertia ixx="0.3" ixy="0.0" ixz="0.0" iyy="0.3" iyz="0.0" izz="0.3"/>
       </inertial>
@@ -218,5 +255,5 @@
       <inertial>
         <origin xyz="0 0 0" rpy="0 0 0"/>
-        <mass value="0.001"/>
+        <mass value="${mass_link8}"/>
         <inertia ixx="0.3" ixy="0.0" ixz="0.0" iyy="0.3" iyz="0.0" izz="0.3"/>
       </inertial>

File: franka_description/robots/panda_arm_model.urdf.xacro (robot description, xacro)
@@ -6,8 +6,8 @@
   <!-- Robot -->
   <xacro:include filename="$(find franka_description)/robots/panda_arm_model.xacro" />
-  <xacro:include filename="$(find franka_description)/robots/panda.gazebo.xacro"/>
+  <xacro:include filename="$(find franka_description)/robots/panda_model.gazebo.xacro"/>
   <xacro:include filename="$(find franka_description)/robots/panda.transmission.xacro"/>
   <xacro:panda_arm xyz = "0 1.5 0"/>
-  <xacro:panda_gazebo robot_name="$(arg robot_name)" />
+  <xacro:panda_model_gazebo robot_name="$(arg robot_name)" />
   <xacro:panda_transmission robot_name="$(arg robot_name)" />
 </robot>

File: franka_description/robots/panda_model.gazebo.xacro (robot description, xacro)
@@ -1,64 +1,73 @@
 <?xml version="1.0"?>
 <robot xmlns:xacro="http://www.ros.org/wiki/xacro">
-    <xacro:macro name="panda_gazebo" params="robot_name">
+    <xacro:macro name="panda_model_gazebo" params="robot_name">
         <!-- Link0 -->
         <gazebo reference="${robot_name}_link0">
-            <mu1>0.61</mu1>
-            <mu2>0.61</mu2>
+            <material>Gazebo/Grey</material>
+            <mu1>0.2</mu1>
+            <mu2>0.2</mu2>
         </gazebo>
         <!-- Link1 -->
         <gazebo reference="${robot_name}_link1">
-            <mu1>0.61</mu1>
-            <mu2>0.61</mu2>
+            <material>Gazebo/White</material>
+            <mu1>0.2</mu1>
+            <mu2>0.2</mu2>
         </gazebo>
         <!-- Link2 -->
         <gazebo reference="${robot_name}_link2">
-            <mu1>0.61</mu1>
-            <mu2>0.61</mu2>
+            <material>Gazebo/White</material>
+            <mu1>0.2</mu1>
+            <mu2>0.2</mu2>
         </gazebo>
         <!-- Link3 -->
         <gazebo reference="${robot_name}_link3">
-            <mu1>0.61</mu1>
-            <mu2>0.61</mu2>
+            <material>Gazebo/White</material>
+            <mu1>0.2</mu1>
+            <mu2>0.2</mu2>
         </gazebo>
         <!-- Link4 -->
         <gazebo reference="${robot_name}_link4">
-            <mu1>0.61</mu1>
-            <mu2>0.61</mu2>
+            <material>Gazebo/White</material>
+            <mu1>0.2</mu1>
+            <mu2>0.2</mu2>
         </gazebo>
         <!-- Link5 -->
         <gazebo reference="${robot_name}_link5">
-            <mu1>0.61</mu1>
-            <mu2>0.61</mu2>
+            <material>Gazebo/White</material>
+            <mu1>0.2</mu1>
+            <mu2>0.2</mu2>
         </gazebo>
         <!-- Link6 -->
         <gazebo reference="${robot_name}_link6">
-            <mu1>0.61</mu1>
-            <mu2>0.61</mu2>
+            <material>Gazebo/White</material>
+            <mu1>0.2</mu1>
+            <mu2>0.2</mu2>
         </gazebo>
         <!-- Link7 -->
         <gazebo reference="${robot_name}_link7">
-            <mu1>0.61</mu1>
-            <mu2>0.61</mu2>
+            <material>Gazebo/White</material>
+            <mu1>0.2</mu1>
+            <mu2>0.2</mu2>
         </gazebo>
         <!-- Link8 -->
         <gazebo reference="${robot_name}_link8">
-            <mu1>0.61</mu1>
-            <mu2>0.61</mu2>
+            <material>Gazebo/White</material>
+            <mu1>0.2</mu1>
+            <mu2>0.2</mu2>
         </gazebo>
         <!-- LinkHand -->
         <gazebo reference="${robot_name}_hand">
-            <mu1>0.61</mu1>
-            <mu2>0.61</mu2>
+            <mu1>0.2</mu1>
+            <mu2>0.2</mu2>
         </gazebo>
         <!-- LinkRightFinger -->
         <gazebo reference="${robot_name}_rightfinger">
-            <mu1>0.61</mu1>
-            <mu2>0.61</mu2>
+            <mu1>0.2</mu1>
+            <mu2>0.2</mu2>
         </gazebo>
         <!-- LinkLeftFinger -->
         <gazebo reference="${robot_name}_leftfinger">
-            <mu1>0.61</mu1>
-            <mu2>0.61</mu2>
+            <mu1>0.2</mu1>
+            <mu2>0.2</mu2>
         </gazebo>
     </xacro:macro>

Commit message: Deleted unnecessary urdf models

File: franka_description/robots/panda_arm.xacro (robot description, xacro)
@@ -1,6 +1,16 @@
 <?xml version='1.0' encoding='utf-8'?>
 <robot xmlns:xacro="http://www.ros.org/wiki/xacro" name="panda">
-  <!-- This masses are incorrect on purpose, off by 20% w.r.t the model-->
-  <xacro:property name="mass_link0" value="3.66357" />
+  <!--Correct masses-->
+  <xacro:property name="mass_link0" value="3.06357" />
+  <xacro:property name="mass_link1" value="2.34471" />
+  <xacro:property name="mass_link2" value="2.36414" />
+  <xacro:property name="mass_link3" value="2.38050" />
+  <xacro:property name="mass_link4" value="2.42754" />
+  <xacro:property name="mass_link5" value="3.49611" />
+  <xacro:property name="mass_link6" value="1.46736" />
+  <xacro:property name="mass_link7" value="0.45606" />
+  <xacro:property name="mass_link8" value="0.001" />
+  <!-- Wrong masses to test adaptability of the algorithms, on purpose off by 20% -->
+  <!--xacro:property name="mass_link0" value="3.66357" />
   <xacro:property name="mass_link1" value="2.04471" />
   <xacro:property name="mass_link2" value="2.56414" />
@@ -10,5 +20,5 @@
   <xacro:property name="mass_link6" value="1.66736" />
   <xacro:property name="mass_link7" value="0.75606" />
-  <xacro:property name="mass_link8" value="0.1" />
+  <xacro:property name="mass_link8" value="0.1" /-->
   <xacro:property name="link0_cog" value="-0.029190 -0.000879 0.056603" />
   <xacro:property name="link1_cog" value="0.000011 -0.031266 -0.069373" />
@@ -19,14 +29,4 @@
   <xacro:property name="link6_cog" value="0.051002 0.006933 0.006169" />
   <xacro:property name="link7_cog" value="0.010361 0.010360 0.079108" />
-  <!-- Correct masses
-  <xacro:property name="mass_link0" value="3.06357" />
-  <xacro:property name="mass_link1" value="2.34471" />
-  <xacro:property name="mass_link2" value="2.36414" />
-  <xacro:property name="mass_link3" value="2.38050" />
-  <xacro:property name="mass_link4" value="2.42754" />
-  <xacro:property name="mass_link5" value="3.49611" />
-  <xacro:property name="mass_link6" value="1.46736" />
-  <xacro:property name="mass_link7" value="0.45606" />
-  <xacro:property name="mass_link8" value="0.001" /> -->
     <xacro:macro name="cylinder_inertial" params="radius length mass *origin">
       <inertial>
@@ -267,16 +267,4 @@
       <dynamics damping="100"/>
     </joint>
-    <!--link name="marker_link">
-    <visual>
-      <geometry>
-          <mesh filename="package://${description_pkg}/meshes/visual/marker.dae" scale="1 1 0.001"/>
-      </geometry>
-    </visual>
-  </link>
-  <joint name="marker_joint" type="fixed">
-    <origin rpy="0 0 0" xyz="0 0 0.0011"/>
-    <parent link="panda_link8"/>
-    <child link="marker_link"/>
-  </joint-->
   </xacro:macro>
 </robot>

File: franka_description/robots/panda_arm_world.urdf.xacro (robot description, xacro)
@@ -6,4 +6,5 @@
   <!-- Robot arm -->
   <xacro:include filename="$(find franka_description)/robots/panda_arm.xacro"/>
+  <xacro:include filename="$(find franka_description)/robots/hand.xacro"/>
   <xacro:include filename="$(find franka_description)/robots/panda.gazebo.xacro"/>
   <xacro:include filename="$(find franka_description)/robots/panda.transmission.xacro"/>
@@ -13,7 +14,4 @@
     <origin xyz="0.3 -0.5 0.0" rpy="0 0 0"/>
   </xacro:robot_pedestal_urdf>
-  <!-- Camera-->
-  <!--xacro:include filename="$(find franka_description)/robots/panda_camera.xacro"/>
-  <xacro:include filename="$(find franka_description)/robots/panda_camera.gazebo.xacro"/-->
   <!-- bins -->
   <xacro:include filename="$(find franka_description)/robots/bin/bin.urdf.xacro"/>
@@ -22,9 +20,8 @@
   <!-- Robot arm definition-->
   <xacro:panda_arm />
+  <!-- Comment or uncomment to add the gripper -->
+  <!--xacro:hand ns="robot1" rpy="0 0 ${-pi/4}" connected_to="panda_link8"/-->
   <xacro:panda_gazebo robot_name="$(arg robot_name)" />
   <xacro:panda_transmission robot_name="$(arg robot_name)" />
-  <!-- Camera definition-->
-  <!--xacro:panda_camera ns="panda" connected_to="world" rpy="0 ${-pi/3} ${pi}" xyz="1 0 0.05"/>
-  <xacro:panda_camera_gazebo /-->
   <!-- pedestal to world -->
   <joint name="robot1_pedestal_to_world_interface" type="fixed">
